Commit message: changed body plan again

File: body.urdf (robot description, URDF)
Before this commit: robot robot, 3 links, 2 joints
Links:
- added link LeftLeg, mass 1; collision box size=0.4 0.4 1; visual box size=0.4 0.4 1
- added link MiddleLeg, mass 1; collision box size=0.2 0.2 0.9; visual box size=0.2 0.2 0.9
- link BackLeg: geometry collision box size=0.4 0.4 1; visual box size=0.4 0.4 1
- link FrontLeg: mass 1 -> 1.8; geometry collision box size=0.4 0.4 0.8; visual box size=0.2 0.2 0.6
- link Torso: geometry collision box size=1 1 0.5; visual box size=1 1 0.5
Joints:
- added joint Torso_LeftLeg: type revolute, parent Torso, child LeftLeg, origin xyz=0.5 -0.5 1 rpy=0 0 0, axis 0 1 0, limit lower=-3.14159 upper=3.14159 effort=0.0 velocity=0.0
- added joint Torso_MiddleLeg: type prismatic, parent Torso, child MiddleLeg, origin xyz=0.25 0 1 rpy=0 0 0, axis 0 0.5 1, limit lower=-0.5 upper=0.5 effort=0.0 velocity=0.0
- joint Torso_BackLeg: origin xyz=1.0 0 1.0 rpy=0 0 0 -> xyz=0.5 0.5 1 rpy=0 0 0
- joint Torso_FrontLeg: origin xyz=2.0 0 1.0 rpy=0 0 0 -> xyz=-0.3 0 1 rpy=0 0 0

Commit message: body plan for testing hidden-neruons

File: body.urdf (robot description, URDF)
Before this commit: robot robot, 5 links, 4 joints
Links:
- added link RightLeg, mass 1; collision box size=0.4 0.4 0.8; visual box size=0.4 0.4 0.8
- link FrontLeg: mass 1.8 -> 1; geometry collision box size=0.4 0.4 0.8; visual box size=0.4 0.4 0.8
Joints:
- added joint Torso_RightLeg: type revolute, parent Torso, child RightLeg, origin xyz=-0.5 -0.5 1 rpy=0 0 0, axis 0 1 0, limit lower=-3.14159 upper=3.14159 effort=0.0 velocity=0.0
- joint Torso_FrontLeg: origin xyz=-0.3 0 1 rpy=0 0 0 -> xyz=-0.5 0.5 1 rpy=0 0 0

Commit message: final body for final project

File: body.urdf (robot description, URDF)
Before this commit: robot robot, 6 links, 5 joints
Links:
- removed link MiddleLeg
- link BackLeg: geometry collision box size=0.5 0.5 0.5; visual box size=0.5 0.5 0.5
- link FrontLeg: geometry collision box size=0.5 0.5 0.5; visual box size=0.5 0.5 0.5
- link LeftLeg: geometry collision box size=0.5 0.5 0.5; visual box size=0.5 0.5 0.5
- link RightLeg: geometry collision box size=0.5 0.5 0.5; visual box size=0.5 0.5 0.5
- link Torso: geometry collision box size=0.5 0.5 0.5; visual box size=0.5 0.5 0.5
Joints:
- removed joint Torso_MiddleLeg
- joint Torso_BackLeg: origin xyz=0.5 0.5 1 rpy=0 0 0 -> xyz=0.25 0 0.5 rpy=0 0 0
- joint Torso_FrontLeg: origin xyz=-0.5 0.5 1 rpy=0 0 0 -> xyz=-25.0 0 0.5 rpy=0 0 0
- joint Torso_LeftLeg: origin xyz=0.5 -0.5 1 rpy=0 0 0 -> xyz=0.25 0 0.5 rpy=0 0 0
- joint Torso_RightLeg: origin xyz=-0.5 -0.5 1 rpy=0 0 0 -> xyz=-0.25 0 0.5 rpy=0 0 0
